Commit message: add slam toolbox

File: description/robot_core.xacro (robot description, xacro)
@@ -18,4 +18,12 @@
     </material>
     <link name="base_link">
+    </link>
+    <!-- BASE_FOOTPRINT -->
+    <joint name="base_footprint_joint" type="fixed">
+        <parent link="base_link"/>
+        <child link="base_footprint"/>
+        <origin xyz="0 0 0" rpy="0 0 0"/>
+    </joint>
+    <link name="base_footprint">
     </link>
     <!-- CHASSIS -->
